Commit message: Integrate Gazebo Harmonic and MoveIt 2 simulation

File: arduinobot_description/urdf/arduinobot_gazebo.xacro (robot description, xacro)
@@ -1,4 +1,10 @@
-<?xml version="1.0"?>
 <robot xmlns:xacro="http://www.ros.org/wiki/xacro" name="arduinobot">
+<!-- Gazebo Harmonic ros2_control plugin -->
+<gazebo>
+  <plugin filename="libgz_ros2_control-system.so"
+          name="gz_ros2_control::GazeboSimROS2ControlPlugin">
+    <parameters>$(find arduinobot_controller)/config/arduinobot_controllers.yaml</parameters>
+  </plugin>
+</gazebo>
     <!-- Gazebo ros2_control plugin -->
     <gazebo>

File: arduinobot_description/urdf/arduinobot_ros2_control.xacro (robot description, xacro)
@@ -3,18 +3,15 @@
     <ros2_control name="RobotSystem" type="system">
         <xacro:property name="PI" value="3.14159265359" />
-        <!-- ros2_control Gazebo -->
-        <xacro:if value="$(arg is_sim)">
-            <hardware>
-                <plugin>gazebo_ros2_control/GazeboSystem</plugin>
-            </hardware>
-            <joint name="joint_5">
-                <param name="mimic">joint_4</param>
-                <param name="multiplier">-1</param>
-                <command_interface name="position">
-                <param name="min">0.0</param>
-                <param name="max">${PI / 2}</param>
-                </command_interface>
-            </joint>
-        </xacro:if>
+        <!-- Gazebo Harmonic ros2_control -->
+<xacro:if value="$(arg is_sim)">
+    <hardware>
+        <plugin>gz_ros2_control/GazeboSimSystem</plugin>
+    </hardware>
+    <joint name="joint_5">
+        <param name="mimic">joint_4</param>
+        <param name="multiplier">-1</param>
+        <state_interface name="position"/>
+    </joint>
+</xacro:if>
         <!-- ros2_control Real Robot -->
         <xacro:unless value="$(arg is_sim)">
